Commit message: Add simplified single leg collision and inertia

File: xacro/leg.xacro (robot description, xacro)
@@ -7,5 +7,5 @@
     <!-- ========================================================= -->
     <link name="${prefix}_hip_motor_fixed">
-      <!-- Fixed hip actuator body: swapped to the other actuator -->
+      <!-- Fixed hip actuator body -->
       <visual>
         <origin xyz="-0.076951 -0.065148 -0.031931" rpy="-1.570796 -0.523599 0"/>
@@ -17,12 +17,15 @@
         <material name="actuator_black"/>
       </visual>
-      <collision>
-        <origin xyz="-0.076951 -0.065148 -0.031931" rpy="-1.570796 -0.523599 0"/>
+      <!-- Simple collision for fixed hip actuator.
+           Origin is at the transformed STL body center, not the mesh origin. -->
+      <collision>
+        <origin xyz="0.000118 -0.083848 0.010078" rpy="-1.570796 -0.523599 0"/>
         <geometry>
           <cylinder radius="0.040" length="0.046"/>
         </geometry>
       </collision>
-      <inertial>
-        <origin xyz="0 0 0" rpy="0 0 0"/>
+      <!-- Approximate inertial values for fixed RobStride actuator -->
+      <inertial>
+        <origin xyz="0.000118 -0.083848 0.010078" rpy="0 0 0"/>
         <mass value="0.405"/>
         <inertia
@@ -87,4 +90,12 @@
         <material name="actuator_black"/>
       </visual>
+      <!-- Simple collision for rotating actuator.
+           Origin is at the transformed STL body center. -->
+      <collision>
+        <origin xyz="-0.000012 0.033700 -0.000153" rpy="-1.570796 0 0"/>
+        <geometry>
+          <cylinder radius="0.040" length="0.046"/>
+        </geometry>
+      </collision>
       <!-- Thigh pulley mount: this rotates about the fixed actuator shaft -->
       <visual>
@@ -107,13 +118,35 @@
         <material name="pulley_orange"/>
       </visual>
-      <!-- Simple collision box for upper-leg physics/debugging -->
-      <collision>
-        <origin xyz="0 0 ${-upper_leg_length/2}" rpy="0 0 0"/>
-        <geometry>
-          <box size="${upper_leg_width} ${upper_leg_depth} ${upper_leg_length}"/>
-        </geometry>
-      </collision>
-      <inertial>
-        <origin xyz="0 0 ${-upper_leg_length/2}" rpy="0 0 0"/>
+                       <!-- Simplified upper-leg side rail collisions.
+           These represent the straight thigh panel areas only.
+           Extended slightly after checking the STEP geometry.
+           The lower cylindrical support/contact center is about 46.125 mm
+           above the bottom of the thigh panel. -->
+      <!-- Left/outer thigh side rail collision -->
+      <collision>
+        <origin xyz="-0.014000 0.071150 -0.0806000" rpy="0 0 0"/>
+        <geometry>
+          <box size="0.008 0.018 0.074"/>
+        </geometry>
+      </collision>
+      <!-- Right/inner thigh side rail collision -->
+      <collision>
+        <origin xyz="0.014000 0.071150 -0.0806000" rpy="0 0 0"/>
+        <geometry>
+          <box size="0.008 0.018 0.074"/>
+        </geometry>
+      </collision>
+      <!-- Small cylindrical lower support/contact approximation.
+           Real support is about 10 mm diameter, so radius is 0.005 m.
+           Center is placed about 46.125 mm above the bottom of the thigh panel. -->
+      <collision>
+        <origin xyz="0.000000 0.071150 -0.151700" rpy="1.570796 0 0"/>
+        <geometry>
+          <cylinder radius="0.005" length="0.045"/>
+        </geometry>
+      </collision>
+      <!-- Approximate inertial values for upper leg assembly -->
+      <inertial>
+        <origin xyz="-0.000015 0.071150 -0.10500" rpy="0 0 0"/>
         <mass value="0.9"/>
         <inertia
@@ -173,13 +206,15 @@
         <material name="pin_yellow"/>
       </visual>
-      <!-- Simple collision box for lower-leg physics/debugging -->
-      <collision>
-        <origin xyz="0 0 ${-lower_leg_length/2}" rpy="0 0 0"/>
-        <geometry>
-          <box size="${lower_leg_width} ${lower_leg_depth} ${lower_leg_length}"/>
-        </geometry>
-      </collision>
-      <inertial>
-        <origin xyz="0 0 ${-lower_leg_length/2}" rpy="0 0 0"/>
+      <!-- Simple collision box for lower leg.
+           Shortened so it stops above the 15 mm foot sphere. -->
+      <collision>
+        <origin xyz="0 0 -0.071" rpy="0 0 0"/>
+        <geometry>
+          <box size="0.026 0.020 0.142"/>
+        </geometry>
+      </collision>
+      <!-- Approximate inertial values for lower leg assembly -->
+      <inertial>
+        <origin xyz="0 0 -0.071" rpy="0 0 0"/>
         <mass value="0.45"/>
         <inertia
@@ -215,4 +250,5 @@
         <material name="foot_red"/>
       </visual>
+      <!-- Simple collision for foot contact -->
       <collision>
         <origin xyz="0 0 0" rpy="0 0 0"/>
@@ -221,4 +257,5 @@
         </geometry>
       </collision>
+      <!-- Approximate inertial values for TPU/rubber foot -->
       <inertial>
         <origin xyz="0 0 0" rpy="0 0 0"/>
