Commit message: Set single leg joint limits and visual colors

File: xacro/const.xacro (robot description, xacro)
@@ -14,8 +14,16 @@
   <xacro:property name="lower_leg_width" value="0.030"/>
   <xacro:property name="lower_leg_depth" value="0.025"/>
-  <!-- Wide RViz-only visualization joint limits -->
+  <!-- Wide RViz-only visualization joint limits.
+       These are not final physical robot limits. -->
   <xacro:property name="hip_lower_limit" value="-3.14159"/>
   <xacro:property name="hip_upper_limit" value="3.14159"/>
-  <xacro:property name="knee_lower_limit" value="-3.14159"/>
-  <xacro:property name="knee_upper_limit" value="3.14159"/>
+  <xacro:property name="knee_lower_limit" value="-.85"/>
+  <xacro:property name="knee_upper_limit" value="3.95"/>
+  <!-- Current knee angle convention:
+       knee_joint = 0 rad is the original CAD/STEP bent pose.
+       knee_joint = +1.570796 rad is approximately the straight-leg pose.
+       Future real-robot angle conversion should use this offset instead
+       of changing mesh origins.
+  -->
+  <xacro:property name="knee_straight_angle" value="1.570796"/>
 </robot>

File: xacro/leg.xacro (robot description, xacro)
@@ -15,5 +15,5 @@
             scale="0.001 0.001 0.001"/>
         </geometry>
-        <material name="joint_black"/>
+        <material name="actuator_black"/>
       </visual>
       <collision>
@@ -55,5 +55,5 @@
             scale="0.001 0.001 0.001"/>
         </geometry>
-        <material name="leg_dark"/>
+        <material name="upper_leg_blue"/>
       </visual>
       <!-- Female thigh panel: flipped inward and aligned flush with male -->
@@ -65,5 +65,5 @@
             scale="0.001 0.001 0.001"/>
         </geometry>
-        <material name="leg_dark"/>
+        <material name="upper_leg_blue"/>
       </visual>
       <!-- Hip shroud -->
@@ -75,5 +75,5 @@
             scale="0.001 0.001 0.001"/>
         </geometry>
-        <material name="joint_black"/>
+        <material name="shroud_purple"/>
       </visual>
       <!-- Rotating actuator attached to thigh pulley mount -->
@@ -85,5 +85,5 @@
             scale="0.001 0.001 0.001"/>
         </geometry>
-        <material name="joint_black"/>
+        <material name="actuator_black"/>
       </visual>
       <!-- Thigh pulley mount: this rotates about the fixed actuator shaft -->
@@ -95,5 +95,5 @@
             scale="0.001 0.001 0.001"/>
         </geometry>
-        <material name="joint_black"/>
+        <material name="shroud_purple"/>
       </visual>
       <!-- 20T motor pulley -->
@@ -105,5 +105,5 @@
             scale="0.001 0.001 0.001"/>
         </geometry>
-        <material name="joint_black"/>
+        <material name="pulley_orange"/>
       </visual>
       <!-- Simple collision box for upper-leg physics/debugging -->
@@ -151,5 +151,5 @@
             scale="0.001 0.001 0.001"/>
         </geometry>
-        <material name="leg_dark"/>
+        <material name="lower_leg_green"/>
       </visual>
       <!-- 30T knee pulley: aligned with lower leg -->
@@ -161,5 +161,5 @@
             scale="0.001 0.001 0.001"/>
         </geometry>
-        <material name="joint_black"/>
+        <material name="pulley_orange"/>
       </visual>
       <!-- Knee pin -->
@@ -171,5 +171,5 @@
             scale="0.001 0.001 0.001"/>
         </geometry>
-        <material name="joint_black"/>
+        <material name="pin_yellow"/>
       </visual>
       <!-- Simple collision box for lower-leg physics/debugging -->
@@ -213,5 +213,5 @@
           <sphere radius="${foot_radius}"/>
         </geometry>
-        <material name="foot_blue"/>
+        <material name="foot_red"/>
       </visual>
       <collision>

File: xacro/materials.xacro (robot description, xacro)
@@ -1,15 +1,27 @@
 <?xml version="1.0"?>
 <robot xmlns:xacro="http://www.ros.org/wiki/xacro">
-<material name="body_gray">
-  <color rgba="1.0 0.0 0.0 1.0"/>
-</material>
-  <material name="leg_dark">
-    <color rgba="0.10 0.10 0.10 1.0"/>
+  <material name="body_gray">
+    <color rgba="0.45 0.45 0.45 1.0"/>
   </material>
-  <material name="joint_black">
+  <material name="actuator_black">
     <color rgba="0.02 0.02 0.02 1.0"/>
   </material>
-  <material name="foot_blue">
-    <color rgba="0.05 0.15 0.80 1.0"/>
+  <material name="upper_leg_blue">
+    <color rgba="0.05 0.20 0.85 1.0"/>
+  </material>
+  <material name="lower_leg_green">
+    <color rgba="0.05 0.65 0.20 1.0"/>
+  </material>
+  <material name="pulley_orange">
+    <color rgba="1.0 0.45 0.05 1.0"/>
+  </material>
+  <material name="pin_yellow">
+    <color rgba="1.0 0.85 0.05 1.0"/>
+  </material>
+  <material name="shroud_purple">
+    <color rgba="0.45 0.10 0.80 1.0"/>
+  </material>
+  <material name="foot_red">
+    <color rgba="0.90 0.05 0.05 1.0"/>
   </material>
 </robot>

Commit message: Add single leg ros2 control position controller

File: xacro/const.xacro (robot description, xacro)
@@ -20,4 +20,14 @@
   <xacro:property name="knee_lower_limit" value="-.85"/>
   <xacro:property name="knee_upper_limit" value="3.95"/>
+  <!-- Actuator/joint effort limits based on RobStride 02 specs.
+     Hip is direct actuator output.
+     Knee uses 30T/20T belt ratio, so torque is multiplied by 1.5.
+       -->
+  <xacro:property name="hip_effort_limit" value="17.0"/>
+  <xacro:property name="knee_effort_limit" value="25.5"/>
+  <!-- Conservative first-pass velocity limits for Gazebo control.
+       These are lower than actuator max speed to keep first control tests stable. -->
+  <xacro:property name="hip_velocity_limit" value="10.0"/>
+  <xacro:property name="knee_velocity_limit" value="10.0"/>
   <!-- Current knee angle convention:
        knee_joint = 0 rad is the original CAD/STEP bent pose.

File: xacro/leg.xacro (robot description, xacro)
@@ -169,5 +169,5 @@
       <origin xyz="0.000118 -0.065148 0.010078" rpy="0 0 0"/>
       <axis xyz="0 1 0"/>
-      <limit lower="${hip_lower_limit}" upper="${hip_upper_limit}" effort="20.0" velocity="10.0"/>
+      <limit lower="${hip_lower_limit}" upper="${hip_upper_limit}" effort="${hip_effort_limit}" velocity="${hip_velocity_limit}"/>
     </joint>
     <!-- ========================================================= -->
@@ -237,5 +237,5 @@
       <origin xyz="-0.000118 0.071450 -0.187578" rpy="0 -1.570796 0"/>
       <axis xyz="0 1 0"/>
-      <limit lower="${knee_lower_limit}" upper="${knee_upper_limit}" effort="20.0" velocity="10.0"/>
+      <limit lower="${knee_lower_limit}" upper="${knee_upper_limit}" effort="${knee_effort_limit}" velocity="${knee_velocity_limit}"/>
     </joint>
     <!-- ========================================================= -->

File: xacro/robot.xacro (robot description, xacro)
@@ -4,4 +4,5 @@
   <xacro:include filename="$(find robot_dog_description)/xacro/materials.xacro"/>
   <xacro:include filename="$(find robot_dog_description)/xacro/leg.xacro"/>
+  <xacro:include filename="$(find robot_dog_description)/xacro/ros2_control.xacro"/>
   <!--
     Single-leg Gazebo/RViz test setup.
@@ -68,3 +69,11 @@
     y="-0.10"
     z="0.24"/>
+  <!-- ROS 2 control interface for Gazebo-controlled single leg -->
+  <xacro:single_leg_ros2_control name="GazeboSimSystem"/>
+  <!-- Gazebo ros2_control plugin -->
+  <gazebo>
+    <plugin filename="gz_ros2_control-system" name="gz_ros2_control::GazeboSimROS2ControlPlugin">
+      <parameters>$(find robot_dog_description)/config/controllers.yaml</parameters>
+    </plugin>
+  </gazebo>
 </robot>

Commit message: Set home pose and vertical rail ground test setup

File: xacro/const.xacro (robot description, xacro)
@@ -14,10 +14,23 @@
   <xacro:property name="lower_leg_width" value="0.030"/>
   <xacro:property name="lower_leg_depth" value="0.025"/>
-  <!-- Wide RViz-only visualization joint limits.
-       These are not final physical robot limits. -->
-  <xacro:property name="hip_lower_limit" value="-3.14159"/>
-  <xacro:property name="hip_upper_limit" value="3.14159"/>
-  <xacro:property name="knee_lower_limit" value="-.85"/>
-  <xacro:property name="knee_upper_limit" value="3.95"/>
+    <!-- Home-relative joint limits.
+       New Gazebo/URDF zero pose is the powered home/squat pose.
+       Hip:
+       Old absolute hip limits were about +/-3.14159 rad.
+       Old home hip was +1.03 rad.
+       New home-relative limits:
+       lower = -3.14159 - 1.03 = -4.17159
+       upper = +3.14159 - 1.03 = +2.11159
+       Knee:
+       Old safe/contact knee range was about -0.80 to +3.90 rad.
+       Old home knee was -0.669 rad.
+       New home-relative limits:
+       lower = -0.80 - (-0.669) = -0.131
+       upper = +3.90 - (-0.669) = +4.569
+  -->
+  <xacro:property name="hip_lower_limit" value="-4.17159"/>
+  <xacro:property name="hip_upper_limit" value="2.11159"/>
+  <xacro:property name="knee_lower_limit" value="-0.131"/>
+  <xacro:property name="knee_upper_limit" value="4.569"/>
   <!-- Actuator/joint effort limits based on RobStride 02 specs.
      Hip is direct actuator output.

File: xacro/leg.xacro (robot description, xacro)
@@ -118,12 +118,10 @@
         <material name="pulley_orange"/>
       </visual>
-                       <!-- Simplified upper-leg side rail collisions.
+      <!-- Simplified upper-leg side rail collisions.
            These represent the straight thigh panel areas only.
-           Extended slightly after checking the STEP geometry.
-           The lower cylindrical support/contact center is about 46.125 mm
-           above the bottom of the thigh panel. -->
+           The 29 mm gap above the lower support cylinder is preserved. -->
       <!-- Left/outer thigh side rail collision -->
       <collision>
-        <origin xyz="-0.014000 0.071150 -0.0806000" rpy="0 0 0"/>
+        <origin xyz="-0.014000 0.071150 -0.080600" rpy="0 0 0"/>
         <geometry>
           <box size="0.008 0.018 0.074"/>
@@ -132,5 +130,5 @@
       <!-- Right/inner thigh side rail collision -->
       <collision>
-        <origin xyz="0.014000 0.071150 -0.0806000" rpy="0 0 0"/>
+        <origin xyz="0.014000 0.071150 -0.080600" rpy="0 0 0"/>
         <geometry>
           <box size="0.008 0.018 0.074"/>
@@ -148,5 +146,5 @@
       <!-- Approximate inertial values for upper leg assembly -->
       <inertial>
-        <origin xyz="-0.000015 0.071150 -0.10500" rpy="0 0 0"/>
+        <origin xyz="-0.000015 0.071150 -0.105000" rpy="0 0 0"/>
         <mass value="0.9"/>
         <inertia
@@ -163,9 +161,13 @@
       Origin is placed on the fixed actuator shaft centerline.
       Axis is Y because the actuator shaft line maps to the URDF Y direction.
+      IMPORTANT HOME CONVENTION:
+      Old squat/home command was hip = +1.03 rad.
+      This offset is now baked into the joint origin so Gazebo/URDF joint
+      value 0.0 starts at the powered home/squat pose.
     -->
     <joint name="${prefix}_hip_joint" type="revolute">
       <parent link="${prefix}_hip_motor_fixed"/>
       <child link="${prefix}_upper_leg"/>
-      <origin xyz="0.000118 -0.065148 0.010078" rpy="0 0 0"/>
+      <origin xyz="0.000118 -0.065148 0.010078" rpy="0 1.03 0"/>
       <axis xyz="0 1 0"/>
       <limit lower="${hip_lower_limit}" upper="${hip_upper_limit}" effort="${hip_effort_limit}" velocity="${hip_velocity_limit}"/>
@@ -229,11 +231,17 @@
     <!--
       Knee joint:
-      Same STEP-derived placement as before, shifted into the new
+      Same STEP-derived placement as before, shifted into the
       hip-joint-centered upper-leg frame.
+      IMPORTANT HOME CONVENTION:
+      Old knee origin pitch was -1.570796.
+      Old squat/home command was knee = -0.669 rad.
+      New pitch = -1.570796 + (-0.669) = -2.239796.
+      This offset is now baked into the joint origin so Gazebo/URDF joint
+      value 0.0 starts at the powered home/squat pose.
     -->
     <joint name="${prefix}_knee_joint" type="revolute">
       <parent link="${prefix}_upper_leg"/>
       <child link="${prefix}_lower_leg"/>
-      <origin xyz="-0.000118 0.071450 -0.187578" rpy="0 -1.570796 0"/>
+      <origin xyz="-0.000118 0.071450 -0.187578" rpy="0 -2.239796 0"/>
       <axis xyz="0 1 0"/>
       <limit lower="${knee_lower_limit}" upper="${knee_upper_limit}" effort="${knee_effort_limit}" velocity="${knee_velocity_limit}"/>

File: xacro/robot.xacro (robot description, xacro)
@@ -6,32 +6,47 @@
   <xacro:include filename="$(find robot_dog_description)/xacro/ros2_control.xacro"/>
   <!--
-    Single-leg Gazebo/RViz test setup.
+    Single-leg Gazebo ground/load test setup.
     This is not the final robot body.
-    It is a temporary fixed test stand so the single leg can be tested
-    in Gazebo before building the full four-leg robot.
+    The gray stand acts like a vertical rail carriage:
+    it can move only up/down so the leg can push against the ground
+    and lift/load the body without the whole model tipping over.
   -->
-  <!-- World reference link for fixed-base Gazebo testing -->
+  <!-- Fixed world reference -->
   <link name="world"/>
-  <!-- Ground/reference frame -->
-  <link name="base_footprint"/>
-  <joint name="world_to_base_footprint" type="fixed">
+  <!-- Sliding carriage reference frame -->
+  <link name="base_footprint">
+    <inertial>
+      <origin xyz="0 0 0" rpy="0 0 0"/>
+      <mass value="0.01"/>
+      <inertia
+        ixx="0.00001"
+        ixy="0.0"
+        ixz="0.0"
+        iyy="0.00001"
+        iyz="0.0"
+        izz="0.00001"/>
+    </inertial>
+  </link>
+  <!--
+    Vertical rail joint:
+    Allows the whole stand/leg assembly to slide only along Z.
+    This lets the leg push the body upward under ground contact.
+  -->
+  <joint name="vertical_rail_joint" type="prismatic">
     <parent link="world"/>
     <child link="base_footprint"/>
     <origin xyz="0 0 0" rpy="0 0 0"/>
+    <axis xyz="0 0 1"/>
+    <limit lower="-0.08" upper="0.60" effort="1000.0" velocity="5.0"/>
+    <dynamics damping="3.0" friction="0.2"/>
   </joint>
-  <!-- Temporary test stand / base fixture -->
+  <!-- Temporary test stand / body carriage -->
   <link name="base_link">
     <!-- Visible test stand block.
-         The front face of this gray box should sit approximately flush
-         with the back face of the fixed black actuator.
-         Measured STEP width from actuator back to shroud front:
-         127.15 mm = 0.12715 m
-         With box y-thickness = 0.08 m:
-         front face y = -0.24655 + 0.04 = -0.20655 m
-    -->
+         Front face is approximately flush with the back face of the fixed actuator. -->
     <visual>
-      <origin xyz="0 -0.24655 0.15" rpy="0 0 0"/>
+      <origin xyz="0 -0.24655 0.21" rpy="0 0 0"/>
       <geometry>
-        <box size="0.24 0.08 0.30"/>
+        <box size="0.24 0.08 0.18"/>
       </geometry>
       <material name="body_gray"/>
@@ -39,13 +54,14 @@
     <!-- Simple collision for test stand -->
     <collision>
-      <origin xyz="0 -0.24655 0.15" rpy="0 0 0"/>
+      <origin xyz="0 -0.24655 0.21" rpy="0 0 0"/>
       <geometry>
-        <box size="0.24 0.08 0.30"/>
+        <box size="0.24 0.08 0.18"/>
       </geometry>
     </collision>
-    <!-- Approximate inertial values for fixed test stand -->
+    <!-- Approximate loaded carriage/body mass.
+         Increase this later to test heavier body loads. -->
     <inertial>
-      <origin xyz="0 -0.24655 0.15" rpy="0 0 0"/>
-      <mass value="5.0"/>
+      <origin xyz="0 -0.24655 0.21" rpy="0 0 0"/>
+      <mass value="2.0"/>
       <inertia
         ixx="0.015"
@@ -62,5 +78,6 @@
     <origin xyz="0 0 0" rpy="0 0 0"/>
   </joint>
-  <!-- Single front-right test leg mounted to the test stand -->
+  <!-- Single front-right test leg mounted to the vertical sliding stand.
+       Current leg zero pose is the home/squat pose. -->
   <xacro:simple_leg
     prefix="front_right"
@@ -68,5 +85,5 @@
     x="0.08"
     y="-0.10"
-    z="0.24"/>
+    z="0.1545"/>
   <!-- ROS 2 control interface for Gazebo-controlled single leg -->
   <xacro:single_leg_ros2_control name="GazeboSimSystem"/>
